Commit message: Began to Add Other Joints
-However realized that the Dorna API and the way I defined my URDF have different coordinate systems. I think I will fix this by creating a new URDF with the Dorna robot in the "all zero" configuration in line with the spec sheets on Dorna's website

File: Dorna_2_URDF/urdf/Dorna_2_URDF.urdf (robot description, URDF)
Before this commit: robot Dorna_2_URDF, 7 links, 6 joints
Joints:
- joint Joint_0: limit lower=-3.1416 upper=2.7925 effort=10 velocity=10.472 -> lower=-2.7925 upper=3.1416 effort=10 velocity=10.472
